File: Ignition.kicad_sch (KiCad schematic)
At the start: 15 parts, among them U10 ITS4200SSJDXUMA1, U11 ITS4200SSJDXUMA1, U12 ITS4200SSJDXUMA1, U13 ITS4200SSJDXUMA1, U9 ITS4200SSJDXUMA1

Commit message: Assigning footprints
Parts:
- C17: renamed from C18; footprint (none) -> Capacitor_SMD:C_0603_1608Metric
- C18: renamed from C17; footprint (none) -> Capacitor_SMD:C_0603_1608Metric
- C19, C20, C21, C22, C23, C24, C25, C26: footprint (none) -> Capacitor_SMD:C_0603_1608Metric
- U10, U11, U12, U13, U9: footprint PG-DSO-8-24_INF -> ITS4200SSJDXUMA1:PG-DSO-8-24_INF
Changed lines of the file:
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@@
       (effects (font (size 1.27 1.27)) (justify right))
     )
-    (property "Footprint" "" (at 174.2948 60.96 0)
+    (property "Footprint" "Capacitor_SMD:C_0603_1608Metric" (at 174.2948 60.96 0)
       (effects (font (size 1.27 1.27)) hide)
     )
@@
       (effects (font (size 1.27 1.27)) (justify right))
     )
-    (property "Footprint" "" (at 80.3148 99.06 0)
+    (property "Footprint" "Capacitor_SMD:C_0603_1608Metric" (at 80.3148 99.06 0)
       (effects (font (size 1.27 1.27)) hide)
     )
@@
       (effects (font (size 1.27 1.27)) (justify right))
     )
-    (property "Footprint" "" (at 80.3148 137.16 0)
+    (property "Footprint" "Capacitor_SMD:C_0603_1608Metric" (at 80.3148 137.16 0)
       (effects (font (size 1.27 1.27)) hide)
     )
@@
       (effects (font (size 1.27 1.27)) (justify right))
     )
-    (property "Footprint" "" (at 126.0348 99.06 0)
+    (property "Footprint" "Capacitor_SMD:C_0603_1608Metric" (at 126.0348 99.06 0)
       (effects (font (size 1.27 1.27)) hide)
     )
@@
       (effects (font (size 1.27 1.27)) (justify right))
     )
-    (property "Footprint" "" (at 220.0148 99.06 0)
+    (property "Footprint" "Capacitor_SMD:C_0603_1608Metric" (at 220.0148 99.06 0)
       (effects (font (size 1.27 1.27)) hide)
     )
@@
       (effects (font (size 1.524 1.524)))
     )
-    (property "Footprint" "PG-DSO-8-24_INF" (at 83.82 127 0)
+    (property "Footprint" "ITS4200SSJDXUMA1:PG-DSO-8-24_INF" (at 83.82 127 0)
       (effects (font (size 1.27 1.27) italic) hide)
     )
@@
       (effects (font (size 1.524 1.524)))
     )
-    (property "Footprint" "PG-DSO-8-24_INF" (at 83.82 50.8 0)
+    (property "Footprint" "ITS4200SSJDXUMA1:PG-DSO-8-24_INF" (at 83.82 50.8 0)
       (effects (font (size 1.27 1.27) italic) hide)
     )
@@
       (effects (font (size 1.27 1.27)) (justify right))
     )
-    (property "Footprint" "" (at 220.0148 60.96 0)
+    (property "Footprint" "Capacitor_SMD:C_0603_1608Metric" (at 220.0148 60.96 0)
       (effects (font (size 1.27 1.27)) hide)
     )
@@
       (effects (font (size 1.524 1.524)))
     )
-    (property "Footprint" "PG-DSO-8-24_INF" (at 177.8 88.9 0)
+    (property "Footprint" "ITS4200SSJDXUMA1:PG-DSO-8-24_INF" (at 177.8 88.9 0)
       (effects (font (size 1.27 1.27) italic) hide)
     )
@@
   (symbol (lib_id "Device:C") (at 127 64.77 180) (unit 1)
     (in_bom yes) (on_board yes) (dnp no) (fields_autoplaced)
-    (property "Reference" "C17" (at 130.81 63.5 0)
+    (property "Reference" "C18" (at 130.81 63.5 0)
       (effects (font (size 1.27 1.27)) (justify right))
     )
@@
       (effects (font (size 1.27 1.27)) (justify right))
     )
-    (property "Footprint" "" (at 126.0348 60.96 0)
+    (property "Footprint" "Capacitor_SMD:C_0603_1608Metric" (at 126.0348 60.96 0)
       (effects (font (size 1.27 1.27)) hide)
     )
@@
       (project "control-module-pcb"
         (path "/4c946e98-79c2-4a2d-bd7f-2a33db8d8c91/01645893-76b1-48ec-a8fc-ebf269c31ffb"
+          (reference "C18") (unit 1)
+        )
+      )
+    )
+  )
+  (symbol (lib_id "power:GND") (at 220.98 109.22 0) (unit 1)
+    (in_bom yes) (on_board yes) (dnp no) (fields_autoplaced)
+    (property "Reference" "#PWR038" (at 220.98 115.57 0)
+      (effects (font (size 1.27 1.27)) hide)
+    )
+    (property "Value" "GND" (at 220.98 114.3 0)
+      (effects (font (size 1.27 1.27)))
+    )
+    (property "Footprint" "" (at 220.98 109.22 0)
+      (effects (font (size 1.27 1.27)) hide)
+    )
+    (property "Datasheet" "" (at 220.98 109.22 0)
+      (effects (font (size 1.27 1.27)) hide)
+    )
+    (pin "1")
+    (instances
+      (project "control-module-pcb"
+        (path "/4c946e98-79c2-4a2d-bd7f-2a33db8d8c91/01645893-76b1-48ec-a8fc-ebf269c31ffb"
+          (reference "#PWR038") (unit 1)
+        )
+      )
+    )
+  )
+  (symbol (lib_id "Device:C") (at 127 140.97 180) (unit 1)
+    (in_bom yes) (on_board yes) (dnp no) (fields_autoplaced)
+    (property "Reference" "C22" (at 130.81 139.7 0)
+      (effects (font (size 1.27 1.27)) (justify right))
+    )
+    (property "Value" "220n" (at 130.81 142.24 0)
+      (effects (font (size 1.27 1.27)) (justify right))
+    )
+    (property "Footprint" "Capacitor_SMD:C_0603_1608Metric" (at 126.0348 137.16 0)
+      (effects (font (size 1.27 1.27)) hide)
+    )
+    (property "Datasheet" "~" (at 127 140.97 0)
+      (effects (font (size 1.27 1.27)) hide)
+    )
+    (pin "1")
+    (pin "2")
+    (instances
+      (project "control-module-pcb"
+        (path "/4c946e98-79c2-4a2d-bd7f-2a33db8d8c91/01645893-76b1-48ec-a8fc-ebf269c31ffb"
+          (reference "C22") (unit 1)
+        )
+      )
+    )
+  )
+  (symbol (lib_id "Device:C") (at 81.28 64.77 180) (unit 1)
+    (in_bom yes) (on_board yes) (dnp no) (fields_autoplaced)
+    (property "Reference" "C17" (at 85.09 63.5 0)
+      (effects (font (size 1.27 1.27)) (justify right))
+    )
+    (property "Value" "1n" (at 85.09 66.04 0)
+      (effects (font (size 1.27 1.27)) (justify right))
+    )
+    (property "Footprint" "Capacitor_SMD:C_0603_1608Metric" (at 80.3148 60.96 0)
+      (effects (font (size 1.27 1.27)) hide)
+    )
+    (property "Datasheet" "~" (at 81.28 64.77 0)
+      (effects (font (size 1.27 1.27)) hide)
+    )
+    (pin "1")
+    (pin "2")
+    (instances
+      (project "control-module-pcb"
+        (path "/4c946e98-79c2-4a2d-bd7f-2a33db8d8c91/01645893-76b1-48ec-a8fc-ebf269c31ffb"
           (reference "C17") (unit 1)
         )
@@
     )
   )
-  (symbol (lib_id "power:GND") (at 220.98 109.22 0) (unit 1)
-    (in_bom yes) (on_board yes) (dnp no) (fields_autoplaced)
-    (property "Reference" "#PWR038" (at 220.98 115.57 0)
-      (effects (font (size 1.27 1.27)) hide)
-    )
-    (property "Value" "GND" (at 220.98 114.3 0)
-      (effects (font (size 1.27 1.27)))
-    )
-    (property "Footprint" "" (at 220.98 109.22 0)
-      (effects (font (size 1.27 1.27)) hide)
-    )
-    (property "Datasheet" "" (at 220.98 109.22 0)
-      (effects (font (size 1.27 1.27)) hide)
-    )
-    (pin "1")
-    (instances
-      (project "control-module-pcb"
-        (path "/4c946e98-79c2-4a2d-bd7f-2a33db8d8c91/01645893-76b1-48ec-a8fc-ebf269c31ffb"
-          (reference "#PWR038") (unit 1)
-        )
-      )
-    )
-  )
-  (symbol (lib_id "Device:C") (at 127 140.97 180) (unit 1)
-    (in_bom yes) (on_board yes) (dnp no) (fields_autoplaced)
-    (property "Reference" "C22" (at 130.81 139.7 0)
-      (effects (font (size 1.27 1.27)) (justify right))
-    )
-    (property "Value" "220n" (at 130.81 142.24 0)
-      (effects (font (size 1.27 1.27)) (justify right))
-    )
-    (property "Footprint" "" (at 126.0348 137.16 0)
-      (effects (font (size 1.27 1.27)) hide)
-    )
-    (property "Datasheet" "~" (at 127 140.97 0)
-      (effects (font (size 1.27 1.27)) hide)
-    )
-    (pin "1")
-    (pin "2")
-    (instances
-      (project "control-module-pcb"
-        (path "/4c946e98-79c2-4a2d-bd7f-2a33db8d8c91/01645893-76b1-48ec-a8fc-ebf269c31ffb"
-          (reference "C22") (unit 1)
-        )
-      )
-    )
-  )
-  (symbol (lib_id "Device:C") (at 81.28 64.77 180) (unit 1)
-    (in_bom yes) (on_board yes) (dnp no) (fields_autoplaced)
-    (property "Reference" "C18" (at 85.09 63.5 0)
-      (effects (font (size 1.27 1.27)) (justify right))
-    )
-    (property "Value" "1n" (at 85.09 66.04 0)
-      (effects (font (size 1.27 1.27)) (justify right))
-    )
-    (property "Footprint" "" (at 80.3148 60.96 0)
-      (effects (font (size 1.27 1.27)) hide)
-    )
-    (property "Datasheet" "~" (at 81.28 64.77 0)
-      (effects (font (size 1.27 1.27)) hide)
-    )
-    (pin "1")
-    (pin "2")
-    (instances
-      (project "control-module-pcb"
-        (path "/4c946e98-79c2-4a2d-bd7f-2a33db8d8c91/01645893-76b1-48ec-a8fc-ebf269c31ffb"
-          (reference "C18") (unit 1)
-        )
-      )
-    )
-  )
   (symbol (lib_id "power:GND") (at 220.98 71.12 0) (unit 1)
     (in_bom yes) (on_board yes) (dnp no) (fields_autoplaced)
@@
       (effects (font (size 1.524 1.524)))
     )
-    (property "Footprint" "PG-DSO-8-24_INF" (at 83.82 88.9 0)
+    (property "Footprint" "ITS4200SSJDXUMA1:PG-DSO-8-24_INF" (at 83.82 88.9 0)
       (effects (font (size 1.27 1.27) italic) hide)
     )
@@
       (effects (font (size 1.27 1.27)) (justify right))
     )
-    (property "Footprint" "" (at 174.2948 99.06 0)
+    (property "Footprint" "Capacitor_SMD:C_0603_1608Metric" (at 174.2948 99.06 0)
       (effects (font (size 1.27 1.27)) hide)
     )
@@
       (effects (font (size 1.524 1.524)))
     )
-    (property "Footprint" "PG-DSO-8-24_INF" (at 177.8 50.8 0)
-      (effects (font (size 1.27 1.27) italic) hide)
-    )
+    (property "Footprint" "ITS4200SSJDXUMA1:PG-DSO-8-24_INF" (at 177.8 50.8 0)
+      (effects (font (size 1.27 1.27) italic) hide)
+    )
