File: Power Outputs.kicad_sch (KiCad schematic)
At the start: 30 parts, among them U4 MIC2039BYM6-TR, U5 MIC2039BYM6-TR, U6 MIC2039BYM6-TR, U7 MIC2039BYM6-TR, U8 MIC2039BYM6-TR

Commit message: Assigning footprints
Parts:
- C10, C11, C12, C13, C14, C15, C16, C7, C8, C9: footprint (none) -> Capacitor_SMD:C_1206_3216Metric
- R10, R11, R12, R13, R14, R15, R16, R17, R2, R33, R34, R35, R36, R8, R9: footprint (none) -> Resistor_SMD:R_0603_1608Metric
- U4, U5, U6, U7, U8: footprint SOT-23-6_M6_MCH -> MIC2039BYM6_TR:SOT-23-6_M6_MCH
Changed lines of the file:
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@@
       (effects (font (size 1.27 1.27)) (justify left))
     )
-    (property "Footprint" "" (at 140.716 147.574 90)
+    (property "Footprint" "Resistor_SMD:R_0603_1608Metric" (at 140.716 147.574 90)
       (effects (font (size 1.27 1.27)) hide)
     )
@@
       (effects (font (size 1.27 1.27)) (justify left))
     )
-    (property "Footprint" "" (at 129.286 183.134 90)
+    (property "Footprint" "Resistor_SMD:R_0603_1608Metric" (at 129.286 183.134 90)
       (effects (font (size 1.27 1.27)) hide)
     )
@@
       (effects (font (size 1.27 1.27)) (justify left))
     )
-    (property "Footprint" "" (at 140.716 112.014 90)
+    (property "Footprint" "Resistor_SMD:R_0603_1608Metric" (at 140.716 112.014 90)
       (effects (font (size 1.27 1.27)) hide)
     )
@@
       (effects (font (size 1.27 1.27)) (justify left))
     )
-    (property "Footprint" "" (at 152.0952 151.13 0)
+    (property "Footprint" "Capacitor_SMD:C_1206_3216Metric" (at 152.0952 151.13 0)
       (effects (font (size 1.27 1.27)) hide)
     )
@@
       (effects (font (size 1.27 1.27)) (justify left))
     )
-    (property "Footprint" "" (at 129.286 147.574 90)
+    (property "Footprint" "Resistor_SMD:R_0603_1608Metric" (at 129.286 147.574 90)
       (effects (font (size 1.27 1.27)) hide)
     )
@@
       (effects (font (size 1.27 1.27)) (justify left))
     )
-    (property "Footprint" "" (at 140.716 76.454 90)
+    (property "Footprint" "Resistor_SMD:R_0603_1608Metric" (at 140.716 76.454 90)
       (effects (font (size 1.27 1.27)) hide)
     )
@@
       (effects (font (size 1.524 1.524)))
     )
-    (property "Footprint" "SOT-23-6_M6_MCH" (at 62.23 172.72 0)
+    (property "Footprint" "MIC2039BYM6_TR:SOT-23-6_M6_MCH" (at 62.23 172.72 0)
       (effects (font (size 1.27 1.27) italic) hide)
     )
@@
       (effects (font (size 1.27 1.27)) (justify left))
     )
-    (property "Footprint" "" (at 152.0952 186.69 0)
+    (property "Footprint" "Capacitor_SMD:C_1206_3216Metric" (at 152.0952 186.69 0)
       (effects (font (size 1.27 1.27)) hide)
     )
@@
       (effects (font (size 1.27 1.27)) (justify left))
     )
-    (property "Footprint" "" (at 140.716 61.214 90)
+    (property "Footprint" "Resistor_SMD:R_0603_1608Metric" (at 140.716 61.214 90)
       (effects (font (size 1.27 1.27)) hide)
     )
@@
       (effects (font (size 1.27 1.27)) (justify left))
     )
-    (property "Footprint" "" (at 140.716 132.334 90)
+    (property "Footprint" "Resistor_SMD:R_0603_1608Metric" (at 140.716 132.334 90)
       (effects (font (size 1.27 1.27)) hide)
     )
@@
       (effects (font (size 1.524 1.524)))
     )
-    (property "Footprint" "SOT-23-6_M6_MCH" (at 62.23 101.6 0)
+    (property "Footprint" "MIC2039BYM6_TR:SOT-23-6_M6_MCH" (at 62.23 101.6 0)
       (effects (font (size 1.27 1.27) italic) hide)
     )
@@
       (effects (font (size 1.27 1.27)) (justify left))
     )
-    (property "Footprint" "" (at 49.2252 76.2 0)
+    (property "Footprint" "Capacitor_SMD:C_1206_3216Metric" (at 49.2252 76.2 0)
       (effects (font (size 1.27 1.27)) hide)
     )
@@
       (effects (font (size 1.27 1.27)) (justify left))
     )
-    (property "Footprint" "" (at 129.286 40.894 90)
+    (property "Footprint" "Resistor_SMD:R_0603_1608Metric" (at 129.286 40.894 90)
       (effects (font (size 1.27 1.27)) hide)
     )
@@
       (effects (font (size 1.27 1.27)) (justify left))
     )
-    (property "Footprint" "" (at 49.2252 182.88 0)
+    (property "Footprint" "Capacitor_SMD:C_1206_3216Metric" (at 49.2252 182.88 0)
       (effects (font (size 1.27 1.27)) hide)
     )
@@
       (effects (font (size 1.27 1.27)) (justify left))
     )
-    (property "Footprint" "" (at 129.286 76.454 90)
+    (property "Footprint" "Resistor_SMD:R_0603_1608Metric" (at 129.286 76.454 90)
       (effects (font (size 1.27 1.27)) hide)
     )
@@
       (effects (font (size 1.27 1.27)) (justify left))
     )
-    (property "Footprint" "" (at 140.716 96.774 90)
+    (property "Footprint" "Resistor_SMD:R_0603_1608Metric" (at 140.716 96.774 90)
       (effects (font (size 1.27 1.27)) hide)
     )
@@
       (effects (font (size 1.27 1.27)) (justify left))
     )
-    (property "Footprint" "" (at 140.716 25.654 90)
+    (property "Footprint" "Resistor_SMD:R_0603_1608Metric" (at 140.716 25.654 90)
       (effects (font (size 1.27 1.27)) hide)
     )
@@
       (effects (font (size 1.27 1.27)) (justify left))
     )
-    (property "Footprint" "" (at 49.2252 40.64 0)
+    (property "Footprint" "Capacitor_SMD:C_1206_3216Metric" (at 49.2252 40.64 0)
       (effects (font (size 1.27 1.27)) hide)
     )
@@
       (effects (font (size 1.524 1.524)))
     )
-    (property "Footprint" "SOT-23-6_M6_MCH" (at 62.23 30.48 0)
+    (property "Footprint" "MIC2039BYM6_TR:SOT-23-6_M6_MCH" (at 62.23 30.48 0)
       (effects (font (size 1.27 1.27) italic) hide)
     )
@@
       (effects (font (size 1.27 1.27)) (justify left))
     )
-    (property "Footprint" "" (at 152.0952 80.01 0)
+    (property "Footprint" "Capacitor_SMD:C_1206_3216Metric" (at 152.0952 80.01 0)
       (effects (font (size 1.27 1.27)) hide)
     )
@@
       (effects (font (size 1.27 1.27)) (justify left))
     )
-    (property "Footprint" "" (at 152.0952 115.57 0)
+    (property "Footprint" "Capacitor_SMD:C_1206_3216Metric" (at 152.0952 115.57 0)
       (effects (font (size 1.27 1.27)) hide)
     )
@@
       (effects (font (size 1.27 1.27)) (justify left))
     )
-    (property "Footprint" "" (at 152.0952 44.45 0)
+    (property "Footprint" "Capacitor_SMD:C_1206_3216Metric" (at 152.0952 44.45 0)
       (effects (font (size 1.27 1.27)) hide)
     )
@@
       (effects (font (size 1.27 1.27)) (justify left))
     )
-    (property "Footprint" "" (at 49.2252 111.76 0)
+    (property "Footprint" "Capacitor_SMD:C_1206_3216Metric" (at 49.2252 111.76 0)
       (effects (font (size 1.27 1.27)) hide)
     )
@@
       (effects (font (size 1.27 1.27)) (justify left))
     )
-    (property "Footprint" "" (at 140.716 40.894 90)
+    (property "Footprint" "Resistor_SMD:R_0603_1608Metric" (at 140.716 40.894 90)
       (effects (font (size 1.27 1.27)) hide)
     )
@@
       (effects (font (size 1.27 1.27)) (justify left))
     )
-    (property "Footprint" "" (at 129.286 112.014 90)
+    (property "Footprint" "Resistor_SMD:R_0603_1608Metric" (at 129.286 112.014 90)
       (effects (font (size 1.27 1.27)) hide)
     )
@@
       (effects (font (size 1.27 1.27)) (justify left))
     )
-    (property "Footprint" "" (at 140.716 183.134 90)
+    (property "Footprint" "Resistor_SMD:R_0603_1608Metric" (at 140.716 183.134 90)
       (effects (font (size 1.27 1.27)) hide)
     )
@@
       (effects (font (size 1.27 1.27)) (justify left))
     )
-    (property "Footprint" "" (at 49.2252 147.32 0)
+    (property "Footprint" "Capacitor_SMD:C_1206_3216Metric" (at 49.2252 147.32 0)
       (effects (font (size 1.27 1.27)) hide)
     )
@@
       (effects (font (size 1.524 1.524)))
     )
-    (property "Footprint" "SOT-23-6_M6_MCH" (at 62.23 137.16 0)
+    (property "Footprint" "MIC2039BYM6_TR:SOT-23-6_M6_MCH" (at 62.23 137.16 0)
       (effects (font (size 1.27 1.27) italic) hide)
     )
@@
       (effects (font (size 1.524 1.524)))
     )
-    (property "Footprint" "SOT-23-6_M6_MCH" (at 62.23 66.04 0)
+    (property "Footprint" "MIC2039BYM6_TR:SOT-23-6_M6_MCH" (at 62.23 66.04 0)
       (effects (font (size 1.27 1.27) italic) hide)
     )
@@
       (effects (font (size 1.27 1.27)) (justify left))
     )
-    (property "Footprint" "" (at 140.716 167.894 90)
-      (effects (font (size 1.27 1.27)) hide)
-    )
+    (property "Footprint" "Resistor_SMD:R_0603_1608Metric" (at 140.716 167.894 90)
+      (effects (font (size 1.27 1.27)) hide)
+    )
